Commit message: (PARTLY BROKEN) - Planning successful but joint rotates in the opposite direction + no commands sent

File: exp-ws/src/single_joint_demo/resources/single-joint-robot/single-joint-demo.urdf (robot description, URDF)
Before this commit: robot single-joint, 3 links, 2 joints
Links:
- removed link base_link
Joints:
- removed joint base_join

Commit message: (FIXED) Joint axes changed to reflect the direction correctly + minor rviz conf file changes

File: exp-ws/src/single_joint_demo/resources/single-joint-robot/single-joint-demo.urdf (robot description, URDF)
Before this commit: robot single-joint-demo-robot, 2 links, 1 joints
Joints:
- joint joint1: axis 0 0 1 -> 0 0 -1
